Commit message: change <gazebo> tag, make the robot move. change the inertial function.

File: src/alpha_description/urdf/alpha.xacro (robot description, xacro)
@@ -16,8 +16,8 @@
     <!-- Constants -->
     <xacro:property name="M_PI" value="3.14159"/>
-    <xacro:property name="left" value="-1"/>
-    <xacro:property name="right" value="1"/>
-    <xacro:property name="back" value="-1"/>
-    <xacro:property name="front" value="1"/>
+    <xacro:property name="left" value="0"/>
+    <xacro:property name="right" value="2"/>
+    <xacro:property name="back" value="0"/>
+    <xacro:property name="front" value="2"/>
     <!-- base link properties -->
     <xacro:property name="base_radius" value="0.5" />
@@ -58,8 +58,27 @@
     <xacro:property name="grasp_frame_radius" value="0.001" />
     <!-- Inertial matrix macro-->
-    <xacro:macro name="inertial_matrix" params="mass">
+    <!-- Macro for inertia matrix -->
+    <xacro:macro name="sphere_inertial_matrix" params="m r">
         <inertial>
-            <mass value="${mass}" />
-            <inertia ixx="1.0" ixy="0.0" ixz="0.0" iyy="0.5" iyz="0.0" izz="1.0" />
+            <mass value="${m}" />
+            <inertia ixx="${2*m*r*r/5}" ixy="0" ixz="0"
+                iyy="${2*m*r*r/5}" iyz="0"
+                izz="${2*m*r*r/5}" />
+        </inertial>
+    </xacro:macro>
+    <xacro:macro name="cylinder_inertial_matrix" params="m r h">
+        <inertial>
+            <mass value="${m}" />
+            <inertia ixx="${m*(3*r*r+h*h)/12}" ixy = "0" ixz = "0"
+                iyy="${m*(3*r*r+h*h)/12}" iyz = "0"
+                izz="${m*r*r/2}" />
+        </inertial>
+    </xacro:macro>
+    <xacro:macro name="box_inertial_matrix" params="m w h d">
+        <inertial>
+            <mass value="${m}" />
+            <inertia ixx="${m*(h*h+d*d)/12}" ixy = "0" ixz = "0"
+                iyy="${m*(w*w+d*d)/12}" iyz = "0"
+                izz="${m*(w*w+h*h)/12}" />
         </inertial>
     </xacro:macro>
@@ -80,5 +99,5 @@
                 </geometry>
             </collision>
-            <xacro:inertial_matrix mass="1"/>
+            <xacro:cylinder_inertial_matrix m="1" r="${link_width}" h="${link_len}"/>
         </link>
         <joint name="joint_${number}" type="revolute">
@@ -92,5 +111,5 @@
     </xacro:macro>
     <!-- motor link and joint macro-->
-    <!-- loc = -1: left;    loc = 1: right  -->
+    <!-- loc = 0: left;    loc = 2: right  -->
     <xacro:macro name="motor_link" params="loc color link_width link_len y_loc z_loc">
         <link name="motor_${loc}" >
@@ -108,10 +127,10 @@
                 </geometry>
             </collision>
-            <xacro:inertial_matrix mass="1"/>
+            <xacro:box_inertial_matrix m="1" w="${link_width}" h="${link_len}" d="${link_width}"/>
         </link>
         <joint name="joint_motor_${loc}" type="fixed">
             <parent link="base_link" />
             <child link="motor_${loc}" />
-            <origin xyz="0 ${loc*y_loc} ${z_loc}" rpy="0 0 0" />
+            <origin xyz="0 ${(loc-1)*y_loc} ${z_loc}" rpy="0 0 0" />
         </joint>
         <gazebo reference="motor_${loc}">
@@ -123,5 +142,5 @@
         <link name="wheel_${loc}" >
             <visual>
-                <origin xyz="0 ${loc*link_len/2} 0" rpy="${M_PI/2} 0 0" />
+                <origin xyz="0 ${(loc-1)*link_len/2} 0" rpy="${M_PI/2} 0 0" />
                 <geometry>
                     <cylinder radius="${link_width}" length="${link_len}"/>
@@ -130,17 +149,18 @@
             </visual>
             <collision>
-                <origin xyz="0 ${loc*link_len/2} 0" rpy="${M_PI/2} 0 0" />
+                <origin xyz="0 ${(loc-1)*link_len/2} 0" rpy="${M_PI/2} 0 0" />
                 <geometry>
                     <cylinder radius="${link_width}" length="${link_len}"/>
                 </geometry>
             </collision>
-            <xacro:inertial_matrix mass="1"/>
+            <xacro:cylinder_inertial_matrix m="1" r="${link_width}" h="${link_len}"/>
         </link>
         <joint name="joint_wheel_${loc}" type="continuous">
             <parent link="motor_${loc}"/>
             <child link="wheel_${loc}"/>
-            <origin xyz="0 ${loc*y_loc} ${z_loc}" rpy="0 0 0" />
-            <axis xyz="0 ${-loc} 0" rpy="0 0" />
-            <dynamics damping="0.7"/>>
+            <origin xyz="0 ${(loc-1)*y_loc} ${z_loc}" rpy="0 0 0" />
+            <axis xyz="0 1 0" rpy="0 0" />
+            <limit effort="100" velocity="100"/>
+            <joint_properties damping="0.0" friction="10.0"/>
         </joint>
         <gazebo reference="wheel_${loc}">
@@ -149,25 +169,25 @@
     </xacro:macro>
     <!-- caster link and joint macro -->
-    <xacro:macro name="caster_link" params="loc color link_width link_len x_loc z_loc">
+    <xacro:macro name="caster_link" params="loc color link_width x_loc z_loc">
         <link name="caster_${loc}" >
             <visual>
                 <origin xyz="0 0 0" rpy="${M_PI/2} 0 0" />
                 <geometry>
-                    <cylinder radius="${link_width}" length="${link_len}"/>
+                    <sphere radius="${link_width}" />
                 </geometry>
                 <material name="${color}" />
             </visual>
             <collision>
-                <origin xyz="0 ${loc*link_len/2} 0" rpy="${M_PI/2} 0 0" />
-                <geometry>
-                    <cylinder radius="${link_width}" length="${link_len}"/>
+                <origin xyz="0 0 0" rpy="0 0 0" />
+                <geometry>
+                    <sphere radius="${link_width}" />
                 </geometry>
             </collision>
-            <xacro:inertial_matrix mass="1"/>
+            <xacro:sphere_inertial_matrix m="1" r="${link_width}"/>
         </link>
         <joint name="joint_caster_${loc}" type="fixed">
             <parent link="base_link"/>
             <child link="caster_${loc}"/>
-            <origin xyz="${loc*x_loc} 0 ${z_loc}" rpy="0 0 0" />
+            <origin xyz="${(loc-1)*x_loc} 0 ${z_loc}" rpy="0 0 0" />
         </joint>
     </xacro:macro>
@@ -180,5 +200,4 @@
             </geometry>
         </visual>
-        <xacro:inertial_matrix mass="0.00001"/>
     </link>
     <joint name="base_footprint_joint" type="fixed">
@@ -190,5 +209,5 @@
     <link name="base_link">
         <visual>
-            <origin xyz="0 0 ${wheel_radius+motor_width+base_len/2}" rpy="0 0 0" />
+            <origin xyz="0 0 ${wheel_radius+motor_width/2+base_len/2}" rpy="0 0 0" />
             <geometry>
                 <cylinder radius="${base_radius}" length="${base_len}"/>
@@ -197,10 +216,10 @@
         </visual>
         <collision>
-            <origin xyz="0 0 ${wheel_radius+motor_width+base_len/2}" rpy="0 0 0" />
+            <origin xyz="0 0 ${wheel_radius+motor_width/2+base_len/2}" rpy="0 0 0" />
             <geometry>
                 <cylinder radius="${base_radius}" length="${base_len}"/>
             </geometry>
         </collision>
-        <xacro:inertial_matrix mass="1"/>
+        <xacro:cylinder_inertial_matrix m="20" r="${base_radius}" h="${base_len}"/>
     </link>
     <!-- motor link -->
@@ -210,6 +229,6 @@
     <wheel_link loc="${left}" color="Blue" link_width="${wheel_radius}" link_len="${wheel_len}" y_loc="${motor_len/2}" z_loc="${-motor_width/2}"/>
     <wheel_link loc="${right}" color="Blue" link_width="${wheel_radius}" link_len="${wheel_len}" y_loc="${motor_len/2}" z_loc="${-motor_width/2}"/>
-    <caster_link loc="${back}" color="Red" link_width="${wheel_radius}" link_len="${wheel_len}" x_loc="${base_radius/2}" z_loc="${wheel_radius}"/>
-    <caster_link loc="${front}" color="Red" link_width="${wheel_radius}" link_len="${wheel_len}" x_loc="${base_radius/2}" z_loc="${wheel_radius}"/>
+    <caster_link loc="${back}" color="Red" link_width="${wheel_radius}" x_loc="${base_radius}" z_loc="${wheel_radius}"/>
+    <caster_link loc="${front}" color="Red" link_width="${wheel_radius}" x_loc="${base_radius}" z_loc="${wheel_radius}"/>
     <!-- arm link -->
     <arm_link parent="base_link" number="1" color="Red" link_width="${link1_width}" link_len="${link1_len}" z_loc="${wheel_radius+motor_width/2+base_len}" axis_x="0" axis_y="0" axis_z="1"/>
@@ -234,5 +253,5 @@
             </geometry>
         </collision>
-        <xacro:inertial_matrix mass="1"/>
+        <xacro:box_inertial_matrix m="1" w="${left_gripper_len}" h="${left_gripper_width}" d="${left_gripper_height}"/>
     </link>
     <link name="gripper_finger_link2">
@@ -250,5 +269,5 @@
             </geometry>
         </collision>
-        <xacro:inertial_matrix mass="1"/>
+        <xacro:box_inertial_matrix m="1" w="${left_gripper_len}" h="${left_gripper_width}" d="${left_gripper_height}"/>
     </link>
     <joint name="finger_joint1" type="prismatic">
@@ -298,8 +317,8 @@
         <material>Gazebo/Blue</material>
     </gazebo>
-    <gazebo reference="caster_-1">
+    <gazebo reference="caster_0">
         <material>Gazebo/Red</material>
     </gazebo>
-    <gazebo reference="caster_1">
+    <gazebo reference="caster_2">
         <material>Gazebo/Red</material>
     </gazebo>
@@ -329,27 +348,27 @@
     <xacro:transmission_block joint_name="joint_5"/>
     <xacro:transmission_block joint_name="joint_6"/>
-    <!-- xacro:transmission_block joint_name="joint_motor_-1"/ -->
-    <!-- xacro:transmission_block joint_name="joint_motor_1"/ -->
-    <!-- xacro:transmission_block joint_name="joint_caster_1"/ -->
-    <!-- xacro:transmission_block joint_name="joint_caster_-1"/ -->
+    <!-- xacro:transmission_block joint_name="joint_motor_0"/ -->
+    <!-- xacro:transmission_block joint_name="joint_motor_2"/ -->
+    <!-- xacro:transmission_block joint_name="joint_caster_2"/ -->
+    <!-- xacro:transmission_block joint_name="joint_caster_0"/ -->
     <xacro:transmission_block joint_name="finger_joint1"/>
     <!-- xacro:transmission_block joint_name="base_footprint_joint"/ -->
-    <transmission name="joint_wheel_1_trans">
+    <transmission name="joint_wheel_2_trans">
         <type>transmission_interface/SimpleTransmission</type>
-        <joint name="joint_wheel_1">
-            <hardwareInterface>hardware_interface/EffortJointInterface</hardwareInterface>
-        </joint>
-        <actuator name="motor_act_1">
-            <hardwareInterface>hardware_interface/EffortJointInterface</hardwareInterface>
+        <joint name="joint_wheel_2">
+            <hardwareInterface>hardware_interface/VelocityJointInterface</hardwareInterface>
+        </joint>
+        <actuator name="motor_act_2">
+            <hardwareInterface>hardware_interface/VelocityJointInterface</hardwareInterface>
             <mechanicalReduction>1</mechanicalReduction>
         </actuator>
     </transmission>
-    <transmission name="joint_wheel_-1_trans">
+    <transmission name="joint_wheel_0_trans">
         <type>transmission_interface/SimpleTransmission</type>
-        <joint name="joint_wheel_-1">
-            <hardwareInterface>hardware_interface/EffortJointInterface</hardwareInterface>
-        </joint>
-        <actuator name="motor_act_-1">
-            <hardwareInterface>hardware_interface/EffortJointInterface</hardwareInterface>
+        <joint name="joint_wheel_0">
+            <hardwareInterface>hardware_interface/VelocityJointInterface</hardwareInterface>
+        </joint>
+        <actuator name="motor_act_0">
+            <hardwareInterface>hardware_interface/VelocityJointInterface</hardwareInterface>
             <mechanicalReduction>1</mechanicalReduction>
         </actuator>
@@ -357,5 +376,10 @@
     <!-- ros_control plugin -->
     <gazebo>
-        <plugin name="differential_drive_controller" filename="libgazebo_ros_diff_plugin.so">
+        <plugin name="gazebo_ros_control" filename="libgazebo_ros_control.so">
+            <robotNamespace>/Alpha</robotNamespace>
+        </plugin>
+    </gazebo>
+    <gazebo>
+        <plugin name="differential_drive_controller" filename="libgazebo_ros_diff_drive.so">
             <rosDebugLevel>Debug</rosDebugLevel>
             <publishWheelTF>true</publishWheelTF>
@@ -366,11 +390,11 @@
             <updateRate>100.0</updateRate>
             <legacyMode>true</legacyMode>
-            <leftJoint>joint_wheel_-1</leftJoint>
-            <rightJoint>joint_wheel_1</rightJoint>
+            <leftJoint>joint_wheel_0</leftJoint>
+            <rightJoint>joint_wheel_2</rightJoint>
             <wheelSeparation>${base_radius*2}</wheelSeparation>
             <wheelDiameter>${2*wheel_radius}</wheelDiameter>
             <broadcastTF>1</broadcastTF>
-            <wheelTorque>30</wheelTorque>
-            <wheelAcceleration>1.8</wheelAcceleration>
+            <wheelTorque>300</wheelTorque>
+            <wheelAcceleration>18</wheelAcceleration>
             <commandTopic>cmd_vel</commandTopic>
             <odometryFrame>odom</odometryFrame>
@@ -379,33 +403,3 @@
         </plugin>
     </gazebo>
-    <!--
-    <gazebo reference="joint_wheel_1">
-        <plugin name="differential_drive_controller" filename="libgazebo_ros_diff_plugin.so">
-            <rosDebugLevel>Debug</rosDebugLevel>
-            <publishWheelTF>true</publishWheelTF>
-            <robotNamespace>/Alpha</robotNamespace>
-            <publishTf>1</publishTf>
-            <publishWheelJointState>true</publishWheelJointState>
-            <alwaysOn>true</alwaysOn>
-            <updateRate>100.0</updateRate>
-            <legacyMode>true</legacyMode>
-            <leftJoint>joint_wheel_-1</leftJoint>
-            <rightJoint>joint_wheel_1</rightJoint>
-            <wheelSeparation>${base_radius*2}</wheelSeparation>
-            <wheelDiameter>${2*wheel_radius}</wheelDiameter>
-            <broadcastTF>1</broadcastTF>
-            <wheelTorque>30</wheelTorque>
-            <wheelAcceleration>1.8</wheelAcceleration>
-            <commandTopic>cmd_vel</commandTopic>
-            <odometryFrame>odom</odometryFrame>
-            <odometryTopic>odom</odometryTopic>
-            <robotBaseFrame>base_footprint</robotBaseFrame>
-        </plugin>
-    </gazebo>
-    -->
-    <gazebo>
-        <plugin name="gazebo_ros_control" filename="libgazebo_ros_control.so">
-            <robotNamespace>/Alpha</robotNamespace>
-        </plugin>
-    </gazebo>
 </robot>

Commit message: 1. Set Moveit! config. 2. add ArbotiX Joint controllers, and provid a trajectory demo py file. 3.change the grippers' location.

File: src/alpha_description/urdf/alpha.xacro (robot description, xacro)
@@ -48,11 +48,11 @@
     <xacro:property name="link6_len" value="0.02" />
     <!-- Left gripper -->
-    <xacro:property name="left_gripper_len" value="0.08" />
+    <xacro:property name="left_gripper_len" value="0.01" />
     <xacro:property name="left_gripper_width" value="0.01" />
-    <xacro:property name="left_gripper_height" value="0.01" />
+    <xacro:property name="left_gripper_height" value="0.08" />
     <!-- Right gripper -->
-    <xacro:property name="right_gripper_len" value="0.08" />
+    <xacro:property name="right_gripper_len" value="0.01" />
     <xacro:property name="right_gripper_width" value="0.01" />
-    <xacro:property name="right_gripper_height" value="0.01" />
+    <xacro:property name="right_gripper_height" value="0.08" />
     <!-- Gripper frame -->
     <xacro:property name="grasp_frame_radius" value="0.001" />
@@ -241,5 +241,5 @@
     <link name="gripper_finger_link1">
         <visual>
-            <origin xyz="0.04 -0.03 0"/>
+            <origin xyz="0 0.03 ${left_gripper_height/2}"/>
             <geometry>
                 <box size="${left_gripper_len} ${left_gripper_width} ${left_gripper_height}" />
@@ -248,5 +248,5 @@
         </visual>
         <collision>
-            <origin xyz="0.04 -0.03 0"/>
+            <origin xyz="0 0.03 ${left_gripper_height/2}"/>
             <geometry>
                 <box size="${left_gripper_len} ${left_gripper_width} ${left_gripper_height}" />
@@ -257,5 +257,5 @@
     <link name="gripper_finger_link2">
         <visual>
-            <origin xyz="0.04 -0.03 0"/>
+            <origin xyz="0 -0.03 ${right_gripper_height/2}"/>
             <geometry>
                 <box size="${right_gripper_len} ${right_gripper_width} ${right_gripper_height}" />
@@ -264,5 +264,5 @@
         </visual>
         <collision>
-            <origin xyz="0.04 -0.03 0"/>
+            <origin xyz="0 -0.03 ${right_gripper_height/2}"/>
             <geometry>
                 <box size="${right_gripper_len} ${right_gripper_width} ${right_gripper_height}" />
@@ -276,5 +276,5 @@
         <origin xyz="0.0 0 ${link6_len}" />
         <axis xyz="0 1 0" />
-        <limit effort="100" lower="0.03" upper="0.06" velocity="1.0"/>
+        <limit effort="100" lower="-0.05" upper="0" velocity="1.0"/>
         <dynamics damping="50" friction="1"/>
     </joint>

Commit message: fixed the ArbotiX can not find "base_l (or r)_wheel_joint".the problam is in the diff_controller.py(Arbotix_ros/arbotix_python/src/arbotix_python)

File: src/alpha_description/urdf/alpha.xacro (robot description, xacro)
@@ -106,5 +106,5 @@
             <origin xyz="0 0 ${z_loc}" rpy="0 0 0" />
             <axis xyz="${axis_x} ${axis_y} ${axis_z}" />
-            <limit effort="300" velocity="1" lower="${-M_PI/2}" upper="${M_PI/2}" />
+            <limit effort="300" velocity="1" lower="${-M_PI}" upper="${M_PI}" />
             <dynamics damping="50" friction="1"/>
         </joint>
@@ -156,15 +156,4 @@
             <xacro:cylinder_inertial_matrix m="1" r="${link_width}" h="${link_len}"/>
         </link>
-        <joint name="joint_wheel_${loc}" type="continuous">
-            <parent link="motor_${loc}"/>
-            <child link="wheel_${loc}"/>
-            <origin xyz="0 ${(loc-1)*y_loc} ${z_loc}" rpy="0 0 0" />
-            <axis xyz="0 1 0" rpy="0 0" />
-            <limit effort="100" velocity="100"/>
-            <joint_properties damping="0.0" friction="10.0"/>
-        </joint>
-        <gazebo reference="wheel_${loc}">
-            <material>Gazebo/Blue</material>
-        </gazebo>
     </xacro:macro>
     <!-- caster link and joint macro -->
@@ -229,4 +218,20 @@
     <wheel_link loc="${left}" color="Blue" link_width="${wheel_radius}" link_len="${wheel_len}" y_loc="${motor_len/2}" z_loc="${-motor_width/2}"/>
     <wheel_link loc="${right}" color="Blue" link_width="${wheel_radius}" link_len="${wheel_len}" y_loc="${motor_len/2}" z_loc="${-motor_width/2}"/>
+    <joint name="base_l_wheel_joint" type="continuous">
+        <parent link="motor_0"/>
+        <child link="wheel_0"/>
+        <origin xyz="0 ${(-1)*motor_len/2} ${-motor_width/2}" rpy="0 0 0" />
+        <axis xyz="0 1 0" rpy="0 0" />
+        <limit effort="100" velocity="100"/>
+        <joint_properties damping="0.0" friction="10.0"/>
+    </joint>
+    <joint name="base_r_wheel_joint" type="continuous">
+        <parent link="motor_2"/>
+        <child link="wheel_2"/>
+        <origin xyz="0 ${motor_len/2} ${-motor_width/2}" rpy="0 0 0" />
+        <axis xyz="0 1 0" rpy="0 0" />
+        <limit effort="100" velocity="100"/>
+        <joint_properties damping="0.0" friction="10.0"/>
+    </joint>
     <caster_link loc="${back}" color="Red" link_width="${wheel_radius}" x_loc="${base_radius}" z_loc="${wheel_radius}"/>
     <caster_link loc="${front}" color="Red" link_width="${wheel_radius}" x_loc="${base_radius}" z_loc="${wheel_radius}"/>
@@ -354,7 +359,7 @@
     <xacro:transmission_block joint_name="finger_joint1"/>
     <!-- xacro:transmission_block joint_name="base_footprint_joint"/ -->
-    <transmission name="joint_wheel_2_trans">
+    <transmission name="base_r_wheel_joint_trans">
         <type>transmission_interface/SimpleTransmission</type>
-        <joint name="joint_wheel_2">
+        <joint name="base_r_wheel_joint">
             <hardwareInterface>hardware_interface/VelocityJointInterface</hardwareInterface>
         </joint>
@@ -364,7 +369,7 @@
         </actuator>
     </transmission>
-    <transmission name="joint_wheel_0_trans">
+    <transmission name="base_l_wheel_joint_trans">
         <type>transmission_interface/SimpleTransmission</type>
-        <joint name="joint_wheel_0">
+        <joint name="base_l_wheel_joint">
             <hardwareInterface>hardware_interface/VelocityJointInterface</hardwareInterface>
         </joint>
@@ -378,4 +383,7 @@
         <plugin name="gazebo_ros_control" filename="libgazebo_ros_control.so">
             <robotNamespace>/Alpha</robotNamespace>
+            <odometryFrame>odom</odometryFrame>
+            <odometryTopic>odom</odometryTopic>
+            <robotBaseFrame>base_footprint</robotBaseFrame>
         </plugin>
     </gazebo>
@@ -390,6 +398,6 @@
             <updateRate>100.0</updateRate>
             <legacyMode>true</legacyMode>
-            <leftJoint>joint_wheel_0</leftJoint>
-            <rightJoint>joint_wheel_2</rightJoint>
+            <leftJoint>base_l_wheel_joint</leftJoint>
+            <rightJoint>base_r_wheel_joint</rightJoint>
             <wheelSeparation>${base_radius*2}</wheelSeparation>
             <wheelDiameter>${2*wheel_radius}</wheelDiameter>
