Commit message: add moveit_pick_and_place_demo.py

File: src/alpha_description/urdf/alpha.xacro (robot description, xacro)
@@ -48,11 +48,11 @@
     <xacro:property name="link6_len" value="0.02" />
     <!-- Left gripper -->
-    <xacro:property name="left_gripper_len" value="0.01" />
+    <xacro:property name="left_gripper_len" value="0.08" />
     <xacro:property name="left_gripper_width" value="0.01" />
-    <xacro:property name="left_gripper_height" value="0.08" />
+    <xacro:property name="left_gripper_height" value="0.01" />
     <!-- Right gripper -->
-    <xacro:property name="right_gripper_len" value="0.01" />
+    <xacro:property name="right_gripper_len" value="0.08" />
     <xacro:property name="right_gripper_width" value="0.01" />
-    <xacro:property name="right_gripper_height" value="0.08" />
+    <xacro:property name="right_gripper_height" value="0.01" />
     <!-- Gripper frame -->
     <xacro:property name="grasp_frame_radius" value="0.001" />
@@ -106,5 +106,5 @@
             <origin xyz="0 0 ${z_loc}" rpy="0 0 0" />
             <axis xyz="${axis_x} ${axis_y} ${axis_z}" />
-            <limit effort="300" velocity="1" lower="${-M_PI}" upper="${M_PI}" />
+            <limit effort="300" velocity="10" lower="${-M_PI}" upper="${M_PI}" />
             <dynamics damping="50" friction="1"/>
         </joint>
@@ -246,5 +246,5 @@
     <link name="gripper_finger_link1">
         <visual>
-            <origin xyz="0 0.03 ${left_gripper_height/2}"/>
+            <origin xyz="${left_gripper_len/2} -0.03 0"/>
             <geometry>
                 <box size="${left_gripper_len} ${left_gripper_width} ${left_gripper_height}" />
@@ -253,5 +253,5 @@
         </visual>
         <collision>
-            <origin xyz="0 0.03 ${left_gripper_height/2}"/>
+            <origin xyz="${left_gripper_len/2} -0.03 0"/>
             <geometry>
                 <box size="${left_gripper_len} ${left_gripper_width} ${left_gripper_height}" />
@@ -262,5 +262,5 @@
     <link name="gripper_finger_link2">
         <visual>
-            <origin xyz="0 -0.03 ${right_gripper_height/2}"/>
+            <origin xyz="${right_gripper_len/2} 0.03 0"/>
             <geometry>
                 <box size="${right_gripper_len} ${right_gripper_width} ${right_gripper_height}" />
@@ -269,5 +269,5 @@
         </visual>
         <collision>
-            <origin xyz="0 -0.03 ${right_gripper_height/2}"/>
+            <origin xyz="${right_gripper_len/2} 0.03 0"/>
             <geometry>
                 <box size="${right_gripper_len} ${right_gripper_width} ${right_gripper_height}" />
@@ -279,7 +279,7 @@
         <parent link="link_6"/>
         <child link="gripper_finger_link1"/>
-        <origin xyz="0.0 0 ${link6_len}" />
+        <origin xyz="0.0 0 ${link6_len}" rpy="${M_PI} ${-M_PI/2} 0"/>
         <axis xyz="0 1 0" />
-        <limit effort="100" lower="-0.05" upper="0" velocity="1.0"/>
+        <limit effort="100" lower="0" upper="0.05" velocity="1.0"/>
         <dynamics damping="50" friction="1"/>
     </joint>
@@ -287,5 +287,5 @@
         <parent link="link_6"/>
         <child link="gripper_finger_link2"/>
-        <origin xyz="0.0 0 ${link6_len}" />
+        <origin xyz="0.0 0 ${link6_len}" rpy="${M_PI} ${-M_PI/2} 0"/>
     </joint>
     <!-- Grasping frame -->
@@ -294,5 +294,5 @@
       <parent link="link_6"/>
       <child link="grasping_frame"/>
-      <origin xyz="0.08 0 0" rpy="0 0 0"/>
+      <origin xyz="0 0 ${link6_len+left_gripper_len}" rpy="${M_PI} ${-M_PI/2} 0"/>
     </joint>
     <!-- ////////////   Gazebo   //////////// -->
@@ -382,7 +382,5 @@
     <gazebo>
         <plugin name="gazebo_ros_control" filename="libgazebo_ros_control.so">
-            <robotNamespace>/Alpha</robotNamespace>
-            <odometryFrame>odom</odometryFrame>
-            <odometryTopic>odom</odometryTopic>
+            <robotNamespace>/alpha</robotNamespace>
             <robotBaseFrame>base_footprint</robotBaseFrame>
         </plugin>
@@ -392,9 +390,9 @@
             <rosDebugLevel>Debug</rosDebugLevel>
             <publishWheelTF>true</publishWheelTF>
-            <robotNamespace>/</robotNamespace>
+            <robotNamespace>/alpha</robotNamespace>
             <publishTf>1</publishTf>
             <publishWheelJointState>true</publishWheelJointState>
             <alwaysOn>true</alwaysOn>
-            <updateRate>100.0</updateRate>
+            <updateRate>50.0</updateRate>
             <legacyMode>true</legacyMode>
             <leftJoint>base_l_wheel_joint</leftJoint>

Commit message: add camera, kinect and laser

File: src/alpha_description/urdf/alpha.xacro (robot description, xacro)
@@ -31,5 +31,5 @@
     <!-- link1 properties -->
     <xacro:property name="link1_width" value="0.03" />
-    <xacro:property name="link1_len" value="0.08" />
+    <xacro:property name="link1_len" value="0.1" />
     <!-- link2 properties -->
     <xacro:property name="link2_width" value="0.03" />
@@ -55,4 +55,18 @@
     <xacro:property name="right_gripper_width" value="0.01" />
     <xacro:property name="right_gripper_height" value="0.01" />
+    <!-- camera -->
+    <xacro:property name="camera_len" value="0.01" />
+    <xacro:property name="camera_width" value="0.03" />
+    <xacro:property name="camera_height" value="0.03" />
+    <!-- kinect -->
+    <xacro:property name="kinect_len" value="0.01" />
+    <xacro:property name="kinect_width" value="0.04" />
+    <xacro:property name="kinect_height" value="0.03" />
+    <!-- laser -->
+    <xacro:property name="laser_width" value="0.025" />
+    <xacro:property name="laser_len" value="0.03" />
+    <!-- platform -->
+    <xacro:property name="platform_width" value="0.005" />
+    <xacro:property name="platform_len" value="0.03" />
     <!-- Gripper frame -->
     <xacro:property name="grasp_frame_radius" value="0.001" />
@@ -163,5 +177,5 @@
                 <origin xyz="0 0 0" rpy="${M_PI/2} 0 0" />
                 <geometry>
-                    <sphere radius="${link_width}" />
+                    <sphere radius="${link_width-0.005}" />
                 </geometry>
                 <material name="${color}" />
@@ -170,5 +184,5 @@
                 <origin xyz="0 0 0" rpy="0 0 0" />
                 <geometry>
-                    <sphere radius="${link_width}" />
+                    <sphere radius="${link_width-0.005}" />
                 </geometry>
             </collision>
@@ -181,4 +195,28 @@
         </joint>
     </xacro:macro>
+    <!-- platform link and joint macro -->
+    <xacro:macro name="platform_link" params="loc x_loc">
+        <link name="platform_${loc}_link">
+            <visual>
+                <origin xyz="0 0 ${platform_len*loc/2}"/>
+                <geometry>
+                    <cylinder radius="${platform_width}" length="${platform_len*loc}"/>
+                </geometry>
+                <material name="White" />
+            </visual>
+            <collision>
+                <origin xyz="0 0 ${platform_len/2}"/>
+                <geometry>
+                    <cylinder radius="${platform_width}" length="${platform_len * loc}"/>
+                </geometry>
+            </collision>
+            <xacro:cylinder_inertial_matrix m="1" r="${platform_width}" h="${platform_len}"/>
+        </link>
+        <joint name="platform_${loc}_joint" type="fixed">
+            <parent link="base_link"/>
+            <child link="platform_${loc}_link"/>
+            <origin xyz="${x_loc} 0 ${wheel_radius+motor_width/2+base_len}" rpy="0 0 0"/>
+        </joint>
+    </xacro:macro>
     <!-- base_footprint is a fictitious link(frame) that is on the ground right below base_link origin -->
     <link name="base_footprint">
@@ -212,4 +250,7 @@
         <xacro:cylinder_inertial_matrix m="20" r="${base_radius}" h="${base_len}"/>
     </link>
+    <!-- platform -->
+    <platform_link loc="1" x_loc="${base_radius-0.03}"/>
+    <platform_link loc="2" x_loc="${base_radius-0.08}"/>
     <!-- motor link -->
     <motor_link loc="${left}" color="Red" link_width="${motor_width}" link_len="${motor_len}" y_loc="${base_radius-motor_len/2}" z_loc="${wheel_radius+motor_width/2}"/>
@@ -222,7 +263,7 @@
         <child link="wheel_0"/>
         <origin xyz="0 ${(-1)*motor_len/2} ${-motor_width/2}" rpy="0 0 0" />
-        <axis xyz="0 1 0" rpy="0 0" />
+        <axis xyz="0 1 0" rpy="0 0 0" />
         <limit effort="100" velocity="100"/>
-        <joint_properties damping="0.0" friction="10.0"/>
+        <joint_properties damping="0.0" friction="0.0"/>
     </joint>
     <joint name="base_r_wheel_joint" type="continuous">
@@ -230,7 +271,7 @@
         <child link="wheel_2"/>
         <origin xyz="0 ${motor_len/2} ${-motor_width/2}" rpy="0 0 0" />
-        <axis xyz="0 1 0" rpy="0 0" />
+        <axis xyz="0 1 0" rpy="0 0 0" />
         <limit effort="100" velocity="100"/>
-        <joint_properties damping="0.0" friction="10.0"/>
+        <joint_properties damping="0.0" friction="0.0"/>
     </joint>
     <caster_link loc="${back}" color="Red" link_width="${wheel_radius}" x_loc="${base_radius}" z_loc="${wheel_radius}"/>
@@ -296,5 +337,79 @@
       <origin xyz="0 0 ${link6_len+left_gripper_len}" rpy="${M_PI} ${-M_PI/2} 0"/>
     </joint>
+    <!-- //////////////////////////////////// -->
+    <!-- ////////////   Sensors  //////////// -->
+    <!-- //////////////////////////////////// -->
+    <link name="camera_link">
+        <visual>
+            <origin xyz="0 0 ${camera_height/2}"/>
+            <geometry>
+                <box size="${camera_len} ${camera_width} ${camera_height}" />
+            </geometry>
+            <material name="White" />
+        </visual>
+        <collision>
+            <origin xyz="0 0 ${camera_height/2}"/>
+            <geometry>
+                <box size="${camera_len} ${camera_width} ${camera_height}" />
+            </geometry>
+        </collision>
+        <xacro:box_inertial_matrix m="1" w="${camera_len}" h="${camera_width}" d="${camera_height}"/>
+    </link>
+    <joint name="camera_joint" type="fixed">
+        <parent link="base_link"/>
+        <child link="camera_link"/>
+        <origin xyz="${base_radius - camera_len} 0 ${wheel_radius+motor_width/2+base_len}" rpy="0 0 0"/>
+    </joint>
+    <link name="kinect_link">
+        <visual>
+            <origin xyz="0 0 ${kinect_height/2}"/>
+            <geometry>
+                <box size="${kinect_len} ${kinect_width} ${kinect_height}" />
+            </geometry>
+            <material name="White" />
+        </visual>
+        <collision>
+            <origin xyz="0 0 ${kinect_height/2}"/>
+            <geometry>
+                <box size="${kinect_len} ${kinect_width} ${kinect_height}" />
+            </geometry>
+        </collision>
+        <xacro:box_inertial_matrix m="1" w="${kinect_len}" h="${kinect_width}" d="${kinect_height}"/>
+    </link>
+    <joint name="kinect_joint" type="fixed">
+        <parent link="platform_1_link"/>
+        <child link="kinect_link"/>
+        <origin xyz="0 0 ${platform_len}" rpy="0 0 0"/>
+    </joint>
+    <joint name="kinect_optical_joint" type="fixed">
+        <origin xyz="0 0 0" rpy="-1.5708 0 -1.5708"/>
+        <parent link="kinect_link"/>
+        <child link="kinect_frame_optical"/>
+    </joint>
+    <link name="kinect_frame_optical"/>
+    <link name="laser_link">
+        <visual>
+            <origin xyz="0 0 ${laser_len/2}"/>
+            <geometry>
+                <cylinder radius="${laser_width}" length="${laser_len}"/>
+            </geometry>
+            <material name="White" />
+        </visual>
+        <collision>
+            <origin xyz="0 0 ${laser_len/2}"/>
+            <geometry>
+                <cylinder radius="${laser_width}" length="${laser_len}"/>
+            </geometry>
+        </collision>
+        <xacro:cylinder_inertial_matrix m="1" r="${laser_width}" h="${laser_len}"/>
+    </link>
+    <joint name="laser_joint" type="fixed">
+        <parent link="platform_2_link"/>
+        <child link="laser_link"/>
+        <origin xyz="0 0 ${platform_len*2}" rpy="0 0 0"/>
+    </joint>
+    <!-- //////////////////////////////////// -->
     <!-- ////////////   Gazebo   //////////// -->
+    <!-- //////////////////////////////////// -->
     <gazebo reference="base_footprint">
         <material>Gazebo/White</material>
@@ -332,4 +447,19 @@
     </gazebo>
     <gazebo reference="gripper_finger_link2">
+        <material>Gazebo/White</material>
+    </gazebo>
+    <gazebo reference="camera_link">
+        <material>Gazebo/Black</material>
+    </gazebo>
+    <gazebo reference="kinect_link">
+        <material>Gazebo/Red</material>
+    </gazebo>
+    <gazebo reference="laser_link">
+        <material>Gazebo/Blue</material>
+    </gazebo>
+    <gazebo reference="platform_1_link">
+        <material>Gazebo/White</material>
+    </gazebo>
+    <gazebo reference="platform_2_link">
         <material>Gazebo/White</material>
     </gazebo>
@@ -353,10 +483,5 @@
     <xacro:transmission_block joint_name="joint_5"/>
     <xacro:transmission_block joint_name="joint_6"/>
-    <!-- xacro:transmission_block joint_name="joint_motor_0"/ -->
-    <!-- xacro:transmission_block joint_name="joint_motor_2"/ -->
-    <!-- xacro:transmission_block joint_name="joint_caster_2"/ -->
-    <!-- xacro:transmission_block joint_name="joint_caster_0"/ -->
     <xacro:transmission_block joint_name="finger_joint1"/>
-    <!-- xacro:transmission_block joint_name="base_footprint_joint"/ -->
     <transmission name="base_r_wheel_joint_trans">
         <type>transmission_interface/SimpleTransmission</type>
@@ -379,4 +504,108 @@
         </actuator>
     </transmission>
+    <!-- Sensors plugin -->
+    <gazebo reference="camera_link">
+        <sensor type="camera" name="camera_node">
+            <update_rate>30.0</update_rate>
+            <camera name="head">
+                <horizontal_fov>1.3962634</horizontal_fov>
+                <image>
+                    <width>1280</width>
+                    <height>720</height>
+                    <format>R8G8B8</format>
+                </image>
+                <clip>
+                    <near>0.02</near>
+                    <far>300</far>
+                </clip>
+                <noise>
+                    <type>gaussian</type>
+                    <mean>0.0</mean>
+                    <stddev>0.007</stddev>
+                </noise>
+            </camera>
+            <plugin name="gazebo_camera" filename="libgazebo_ros_camera.so">
+                <alwaysOn>true</alwaysOn>
+                <updateRate>0.0</updateRate>
+                <cameraName>/camera</cameraName>
+                <imageTopicName>image_raw_camera</imageTopicName>
+                <cameraInfoTopicName>camera_info</cameraInfoTopicName>
+                <frameName>camera_link</frameName>
+                <hackBaseline>0.07</hackBaseline>
+                <distortionK1>0.0</distortionK1>
+                <distortionK2>0.0</distortionK2>
+                <distortionK3>0.0</distortionK3>
+                <distortionT1>0.0</distortionT1>
+                <distortionT2>0.0</distortionT2>
+            </plugin>
+        </sensor>
+    </gazebo>
+    <gazebo reference="laser_link">
+        <sensor type="ray" name="rplidar">
+            <pose>0 0 0 0 0 0</pose>
+            <visualize>false</visualize>
+            <update_rate>5.5</update_rate>
+            <ray>
+                <scan>
+                  <horizontal>
+                    <samples>360</samples>
+                    <resolution>1</resolution>
+                    <min_angle>-3</min_angle>
+                    <max_angle>3</max_angle>
+                  </horizontal>
+                </scan>
+                <range>
+                  <min>0.10</min>
+                  <max>6.0</max>
+                  <resolution>0.01</resolution>
+                </range>
+                <noise>
+                    <type>gaussian</type>
+                  <mean>0.0</mean>
+                  <stddev>0.01</stddev>
+                </noise>
+            </ray>
+            <plugin name="gazebo_rplidar" filename="libgazebo_ros_laser.so">
+                <topicName>/scan</topicName>
+                <frameName>laser_link</frameName>
+            </plugin>
+        </sensor>
+    </gazebo>
+    <gazebo reference="kinect_link">
+        <sensor type="depth" name="camera">
+            <always_on>true</always_on>
+            <update_rate>20.0</update_rate>
+            <camera>
+                <horizontal_fov>${60.0*M_PI/180.0}</horizontal_fov>
+                <image>
+                    <format>R8G8B8</format>
+                    <width>640</width>
+                    <height>480</height>
+                </image>
+                <clip>
+                    <near>0.05</near>
+                    <far>8.0</far>
+                </clip>
+            </camera>
+            <plugin name="kinect_camare_controller" filename="libgazebo_ros_openni_kinect.so">
+                <cameraName>kinect</cameraName>
+                <alwaysOn>true</alwaysOn>
+                <updateRate>10</updateRate>
+                <imageTopicName>rgb/image_raw</imageTopicName>
+                <depthImageTopicName>depth/image_raw_kinect</depthImageTopicName>
+                <pointCloudTopicName>depth/points</pointCloudTopicName>
+                <cameraInfoTopicName>rgb/camera_info</cameraInfoTopicName>
+                <depthImageCameraInfoTopicName>depth/camera_info</depthImageCameraInfoTopicName>
+                <frameName>kinect_frame_optical</frameName>
+                <baseline>0.1</baseline>
+                <distortion_k1>0.0</distortion_k1>
+                <distortion_k2>0.0</distortion_k2>
+                <distortion_k3>0.0</distortion_k3>
+                <distortion_t1>0.0</distortion_t1>
+                <distortion_t2>0.0</distortion_t2>
+                <pointCloudCutoff>0.4</pointCloudCutoff>
+            </plugin>
+        </sensor>
+    </gazebo>
     <!-- ros_control plugin -->
     <gazebo>
